Commit message: move over the xacro file (maybe later move over the base urdf too)

File: models/ur5e_robot.urdf (robot description, URDF)
Before this commit: robot ur5e, 13 links, 12 joints
Links:
- added link base
- added link camera_bottom_screw_frame
- added link camera_color_frame
- added link camera_color_optical_frame
- added link camera_depth_frame
- added link camera_depth_optical_frame
- added link camera_left_ir_frame
- added link camera_left_ir_optical_frame
- added link camera_link, mass 0.564; collision box size=0.02505 0.09 0.025; visual mesh filename=package://realsense2_camera/meshes/d435.dae
- added link camera_right_ir_frame
- added link camera_right_ir_optical_frame
- added link grasp_point_fixed
- added link tool0
Joints:
- added joint base_link-base_fixed_joint: type fixed, parent base_link, child base, origin xyz=0 0 0 rpy=0 0 -3.14159265359
- added joint camera_color_joint: type fixed, parent camera_depth_frame, child camera_color_frame, origin xyz=0 0.015 0 rpy=0 0 0
- added joint camera_color_optical_joint: type fixed, parent camera_color_frame, child camera_color_optical_frame, origin xyz=0 0 0 rpy=-1.57079632679 0 -1.57079632679
- added joint camera_depth_joint: type fixed, parent camera_link, child camera_depth_frame, origin xyz=0 0 0 rpy=0 0 0
- added joint camera_depth_optical_joint: type fixed, parent camera_depth_frame, child camera_depth_optical_frame, origin xyz=0 0 0 rpy=-1.57079632679 0 -1.57079632679
- added joint camera_joint: type fixed, parent camera_holder, child camera_bottom_screw_frame, origin xyz=0 0.02 -0.049 rpy=0 -2.18139632679 -1.57079632679
- added joint camera_left_ir_joint: type fixed, parent camera_depth_frame, child camera_left_ir_frame, origin xyz=0 0.0 0 rpy=0 0 0
- added joint camera_left_ir_optical_joint: type fixed, parent camera_left_ir_frame, child camera_left_ir_optical_frame, origin xyz=0 0 0 rpy=-1.57079632679 0 -1.57079632679
- added joint camera_link_joint: type fixed, parent camera_bottom_screw_frame, child camera_link, origin xyz=0 0.0175 0.0125 rpy=0 0 0
- added joint camera_right_ir_joint: type fixed, parent camera_depth_frame, child camera_right_ir_frame, origin xyz=0 -0.05 0 rpy=0 0 0
- added joint camera_right_ir_optical_joint: type fixed, parent camera_right_ir_frame, child camera_right_ir_optical_frame, origin xyz=0 0 0 rpy=-1.57079632679 0 -1.57079632679
- added joint grasp_point_fixed_joint: type fixed, parent hand_link, child grasp_point_fixed, origin xyz=0.0 0.061 0.0 rpy=0.0 0.0 -1.57079632679
- added joint wrist_3_link-tool0_fixed_joint: type fixed, parent wrist_3_link, child tool0, origin xyz=0 0.1 0 rpy=-1.57079632679 0 0
- joint camera_holder_fixed_joint: origin xyz=0.0 0.0 0.0 rpy=0.0 0.0 0.0 -> xyz=0.0315 -0.001 0.0 rpy=-1.57079632679 -1.57079632679 0.0; parent wrist_3_link -> hand_link
- joint finger_l_fixed_joint: origin xyz=0.0 0.061 0.0 rpy=0.0 0.0 -1.57079632679 -> xyz=0.0 0.0 0.0 rpy=0.0 0.0 0.0; parent hand_link -> grasp_point_fixed
- joint finger_r_fixed_joint: origin xyz=0.0 0.061 0.0 rpy=3.14159265359 0.0 -1.57079632679 -> xyz=0.0 0.0 0.0 rpy=3.14159265359 0.0 0.0; parent hand_link -> grasp_point_fixed

Commit message: add copies from other packages

File: models/ur5e_robot.urdf (robot description, URDF)
Before this commit: robot ur5e, 26 links, 25 joints
Links:
- removed link base
- removed link ee_link
- removed link grasp_point_fixed
- removed link tool0
Joints:
- removed joint base_link-base_fixed_joint
- removed joint ee_fixed_joint
- removed joint grasp_point_fixed_joint
- removed joint wrist_3_link-tool0_fixed_joint
- joint finger_l_fixed_joint: axis (none) -> 0 0 1; limit (none) -> lower=0 upper=0.020 effort=150.0 velocity=1.0; origin xyz=0.0 0.0 0.0 rpy=0.0 0.0 0.0 -> xyz=0.0 0.061 -0.0059 rpy=0.0 0.0 -1.57079632679; parent grasp_point_fixed -> hand_link; type fixed -> prismatic
- joint finger_r_fixed_joint: axis (none) -> 0 0 1; limit (none) -> lower=0 upper=0.020 effort=150.0 velocity=1.0; origin xyz=0.0 0.0 0.0 rpy=3.14159265359 0.0 0.0 -> xyz=0.0 0.061 0.0059 rpy=3.14159265359 0.0 -1.57079632679; parent grasp_point_fixed -> hand_link; type fixed -> prismatic

File: models/ur5e_robot.urdf.xacro (robot description, xacro)
@@ -3,5 +3,5 @@
        name="ur5e" >
   <!-- ur5e -->
-  <xacro:include filename="$(find ur_e_description)/urdf/ur5e.urdf.xacro" />
+  <xacro:include filename="$(find vrep_ur5_ros)/urdf/ur5e.urdf.xacro" />
   <!-- arm -->
   <xacro:ur5e_robot prefix="" joint_limited="false"/>
