Commit message: after loading urdf in vrep, you just have to activate joints and add camera

File: models/_d435.urdf.xacro (robot description, xacro)
@@ -5,4 +5,5 @@
 This is the URDF model for the Intel RealSense 430 camera, in it's
 aluminum peripherial evaluation case.
+copied and modified from https://github.com/intel-ros/realsense
 -->
 <robot name="sensor_d435" xmlns:xacro="http://ros.org/wiki/xacro">
@@ -33,15 +34,9 @@
       <xacro:insert_block name="origin" />
       <parent link="${parent}"/>
-      <child link="camera_bottom_screw_frame" />
-    </joint>
-    <link name="camera_bottom_screw_frame"/>
-    <joint name="camera_link_joint" type="fixed">
-      <origin xyz="0 ${d435_cam_depth_py} ${d435_cam_depth_pz}" rpy="0 0 0"/>
-      <parent link="camera_bottom_screw_frame"/>
       <child link="camera_link" />
     </joint>
     <link name="camera_link">
       <visual>
-      <origin xyz="${d435_cam_mount_from_center_offset} ${-d435_cam_depth_py} 0" rpy="${M_PI/2} 0 ${M_PI/2}"/>
+      <origin xyz="${d435_cam_mount_from_center_offset} ${-d435_cam_depth_py + d435_cam_depth_py} ${d435_cam_depth_pz}" rpy="${M_PI/2} 0 ${M_PI/2}"/>
         <geometry>
           <!-- <box size="${d435_cam_width} ${d435_cam_height} ${d435_cam_depth}"/> -->
@@ -52,5 +47,5 @@
       </visual>
       <collision>
-        <origin xyz="0 ${-d435_cam_depth_py} 0" rpy="0 0 0"/>
+        <origin xyz="0 ${-d435_cam_depth_py + d435_cam_depth_py} ${d435_cam_depth_pz}" rpy="0 0 0"/>
         <geometry>
         <box size="${d435_cam_depth} ${d435_cam_width} ${d435_cam_height}"/>
@@ -64,47 +59,8 @@
       </inertial>
     </link>
-    <!-- camera depth joints and links -->
-    <joint name="camera_depth_joint" type="fixed">
-      <origin xyz="0 0 0" rpy="0 0 0"/>
-      <parent link="camera_link"/>
-      <child link="camera_depth_frame" />
-    </joint>
-    <link name="camera_depth_frame"/>
-    <joint name="camera_depth_optical_joint" type="fixed">
-      <origin xyz="0 0 0" rpy="${-M_PI/2} 0 ${-M_PI/2}" />
-      <parent link="camera_depth_frame" />
-      <child link="camera_depth_optical_frame" />
-    </joint>
-    <link name="camera_depth_optical_frame"/>
-    <!-- camera left IR joints and links -->
-    <joint name="camera_left_ir_joint" type="fixed">
-      <origin xyz="0 ${d435_cam_depth_to_left_ir_offset} 0" rpy="0 0 0" />
-      <parent link="camera_depth_frame" />
-      <child link="camera_left_ir_frame" />
-    </joint>
-    <link name="camera_left_ir_frame"/>
-    <joint name="camera_left_ir_optical_joint" type="fixed">
-      <origin xyz="0 0 0" rpy="${-M_PI/2} 0 ${-M_PI/2}" />
-      <parent link="camera_left_ir_frame" />
-      <child link="camera_left_ir_optical_frame" />
-    </joint>
-    <link name="camera_left_ir_optical_frame"/>
-    <!-- camera right IR joints and links -->
-    <joint name="camera_right_ir_joint" type="fixed">
-      <origin xyz="0 ${d435_cam_depth_to_right_ir_offset} 0" rpy="0 0 0" />
-      <parent link="camera_depth_frame" />
-      <child link="camera_right_ir_frame" />
-    </joint>
-    <link name="camera_right_ir_frame"/>
-    <joint name="camera_right_ir_optical_joint" type="fixed">
-      <origin xyz="0 0 0" rpy="${-M_PI/2} 0 ${-M_PI/2}" />
-      <parent link="camera_right_ir_frame" />
-      <child link="camera_right_ir_optical_frame" />
-    </joint>
-    <link name="camera_right_ir_optical_frame"/>
     <!-- camera color joints and links -->
     <joint name="camera_color_joint" type="fixed">
       <origin xyz="0 ${d435_cam_depth_to_color_offset} 0" rpy="0 0 0" />
-      <parent link="camera_depth_frame" />
+      <parent link="camera_link" />
       <child link="camera_color_frame" />
     </joint>

File: models/ur5e.urdf.xacro (robot description, xacro)
@@ -1,3 +1,6 @@
 <?xml version="1.0"?>
+<!--
+Copied and modified from https://github.com/dniewinski/universal_robot
+-->
 <robot xmlns:xacro="http://ros.org/wiki/xacro">
   <xacro:include filename="$(find ur_e_description)/urdf/ur.transmission.xacro" />
@@ -410,5 +413,5 @@
     <xacro:ur_arm_gazebo prefix="${prefix}" />
     <!-- realsense camera -->
-    <xacro:include filename="$(find vrep_ur5_ros)/urdf/_d435.urdf.xacro" />
+    <xacro:include filename="$(find vrep_ur5_ros)/models/_d435.urdf.xacro" />
     <!-- see http://wiki.ros.org/xacro for an explanation of the syntax of starred parameter passing -->
     <xacro:sensor_d435 parent="${prefix}camera_holder">

File: models/ur5e_robot.urdf (robot description, URDF)
Before this commit: robot ur5e, 22 links, 21 joints
Links:
- removed link camera_bottom_screw_frame
- removed link camera_depth_frame
- removed link camera_depth_optical_frame
- removed link camera_left_ir_frame
- removed link camera_left_ir_optical_frame
- removed link camera_right_ir_frame
- removed link camera_right_ir_optical_frame
Joints:
- removed joint camera_depth_joint
- removed joint camera_depth_optical_joint
- removed joint camera_left_ir_joint
- removed joint camera_left_ir_optical_joint
- removed joint camera_link_joint
- removed joint camera_right_ir_joint
- removed joint camera_right_ir_optical_joint
- joint camera_color_joint: parent camera_depth_frame -> camera_link
- joint camera_joint: child camera_bottom_screw_frame -> camera_link

File: models/ur5e_robot.urdf.xacro (robot description, xacro)
@@ -3,5 +3,5 @@
        name="ur5e" >
   <!-- ur5e -->
-  <xacro:include filename="$(find vrep_ur5_ros)/urdf/ur5e.urdf.xacro" />
+  <xacro:include filename="$(find vrep_ur5_ros)/models/ur5e.urdf.xacro" />
   <!-- arm -->
   <xacro:ur5e_robot prefix="" joint_limited="false"/>
