Commit message: fix camera alignment because i moved the joint before for ease of vrep upload

File: urdf/_d435.urdf.xacro (robot description, xacro)
@@ -61,5 +61,5 @@
     <!-- camera color joints and links -->
     <joint name="camera_color_joint" type="fixed">
-      <origin xyz="0 ${d435_cam_depth_to_color_offset} 0" rpy="0 0 0" />
+      <origin xyz="0 ${d435_cam_depth_to_color_offset + d435_cam_depth_py} ${d435_cam_depth_pz}" rpy="0 0 0" />
       <parent link="camera_link" />
       <child link="camera_color_frame" />

File: urdf/ur5e.urdf.xacro (robot description, xacro)
@@ -413,5 +413,5 @@
     <xacro:ur_arm_gazebo prefix="${prefix}" />
     <!-- realsense camera -->
-    <xacro:include filename="$(find vrep_ur5_ros)/models/_d435.urdf.xacro" />
+    <xacro:include filename="$(find vrep_ur5_ros)/urdf/_d435.urdf.xacro" />
     <!-- see http://wiki.ros.org/xacro for an explanation of the syntax of starred parameter passing -->
     <xacro:sensor_d435 parent="${prefix}camera_holder">

File: urdf/ur5e_robot.urdf (robot description, URDF)
Before this commit: robot ur5e, 15 links, 14 joints
Joints:
- joint camera_color_joint: origin xyz=0 0.015 0 rpy=0 0 0 -> xyz=0 0.0325 0.0125 rpy=0 0 0

File: urdf/ur5e_robot.urdf.xacro (robot description, xacro)
@@ -3,5 +3,5 @@
        name="ur5e" >
   <!-- ur5e -->
-  <xacro:include filename="$(find vrep_ur5_ros)/models/ur5e.urdf.xacro" />
+  <xacro:include filename="$(find vrep_ur5_ros)/urdf/ur5e.urdf.xacro" />
   <!-- arm -->
   <xacro:ur5e_robot prefix="" joint_limited="false"/>
