Commit message: this seems correctly simulating (though feels a little slow)

File: urdf/ur5e.urdf.xacro (robot description, xacro)
@@ -371,5 +371,5 @@
       </xacro:cylinder_inertial>
     </link>
-    <joint name="${prefix}finger_l_fixed_joint" type="prismatic">
+    <joint name="${prefix}finger_l_joint" type="prismatic">
       <parent link="${prefix}hand_link" />
       <child link = "${prefix}finger_l_link" />
@@ -379,5 +379,5 @@
       <axis xyz="0 0 1"/>
     </joint>
-    <joint name="${prefix}finger_r_fixed_joint" type="prismatic">
+    <joint name="${prefix}finger_r_joint" type="prismatic">
       <parent link="${prefix}hand_link" />
       <child link = "${prefix}finger_r_link" />
